File: hw/kicad_schematics/CIRCLE.kicad_sch (KiCad schematic)
At the start: 10 parts

Commit message: Filled infos on Schematics
Other:
- company: (none) -> Cyberpunk.company
- title: (none) -> CoolKid'sBadge
Changed lines of the file:
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@@
 	(generator_version "8.0")
 	(paper "A4")
+	(title_block
+		(title "CoolKid'sBadge")
+		(date "2024-07-31")
+		(rev "1.1")
+		(company "Cyberpunk.company")
+		(comment 1 "Electronic Conference badge created for LeHack2024 - by Tixlegeek")
+		(comment 2 "https://cyberpunk.company")
+		(comment 3 "https://tixlegeek.io/splash")
+	)
 	(wire
 		(pts
