File: hw/kicad_schematics/CoolKidsBadge.kicad_sch (KiCad schematic)
At the start: 56 parts, among them J1 USB_C_Receptacle_USB2.0_16P, J4 Conn_01x08_Pin, J5 Conn_01x10_Pin, Q5 UMH3N, SW1 BOOT, SW2 RESET, U1 ESP32-S3-WROOM-1, U2 NRF24L01_SMD, U3 AMS1117-3.3, U4 CH340C

Commit message: Filled infos on Schematics
Other:
- company: (none) -> Cyberpunk.company
- title: (none) -> CoolKid'sBadge
Changed lines of the file:
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@@
 	(generator_version "8.0")
 	(paper "A4")
+	(title_block
+		(title "CoolKid'sBadge")
+		(date "2024-07-31")
+		(rev "1.1")
+		(company "Cyberpunk.company")
+		(comment 1 "Electronic Conference badge created for LeHack2024 - by Tixlegeek")
+		(comment 2 "https://cyberpunk.company")
+		(comment 3 "https://tixlegeek.io/splash")
+	)
 	(junction
 		(at 238.76 142.24)
